File: PCB KiCad/DRS DIP/DRS.kicad_pcb (KiCad board)
At the start: 2 copper layers, 97.5 x 82.5 mm, 62 parts, among them J1 Jp7, J2 Jp8, J3 Jp8, J4 Conn_02x05_Odd_Even, SW1 SW_Push, SW2 SW_Push, SW3 SW_Push, U1 ATmega8-16PU, U2 LM2596S-ADJ, U3 LM2596S-ADJ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

Commit message: 04_14 CANv2
Other:
- net class Default: clearance 0.2 -> 0.5; trace_width 0.25 -> 0.5
- rule trace_clearance: 0.2 -> 0.5
- rule trace_min: 0.2 -> 0.5
Changed lines of the file:
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@@
   )
   (setup
-    (last_trace_width 0.75)
+    (last_trace_width 0.5)
     (user_trace_width 0.5)
     (user_trace_width 0.75)
     (user_trace_width 1)
     (user_trace_width 2)
-    (trace_clearance 0.2)
+    (trace_clearance 0.5)
     (zone_clearance 0.508)
     (zone_45_only no)
-    (trace_min 0.2)
+    (trace_min 0.5)
     (via_size 0.8)
     (via_drill 0.4)
@@
   (net 31 "Net-(D1-Pad1)")
   (net_class Default "To jest domyślna klasa połączeń."
-    (clearance 0.2)
-    (trace_width 0.25)
+    (clearance 0.5)
+    (trace_width 0.5)
     (via_dia 0.8)
     (via_drill 0.4)
     (uvia_dia 0.3)
     (uvia_drill 0.1)
+    (diff_pair_width 0.5)
+    (diff_pair_gap 0.25)
     (add_net +12P)
     (add_net +12V)
@@
   (segment (start 37.2 71.2) (end 36 71.2) (width 1) (layer F.Cu) (net 1))
   (segment (start 38 72) (end 37.2 71.2) (width 1) (layer F.Cu) (net 1))
-  (segment (start 38 77) (end 38 80) (width 1) (layer F.Cu) (net 1))
-  (segment (start 27.6 103.4) (end 27.6 105) (width 0.75) (layer F.Cu) (net 1))
-  (segment (start 39 92) (end 27.6 103.4) (width 0.75) (layer F.Cu) (net 1))
-  (segment (start 38 80) (end 39 81) (width 0.75) (layer F.Cu) (net 1))
-  (segment (start 39 81) (end 39 92) (width 0.75) (layer F.Cu) (net 1))
+  (segment (start 38 80) (end 39 81) (width 0.75) (layer F.Cu) (net 1) (status 1000000))
+  (segment (start 39 81) (end 39 92) (width 0.75) (layer F.Cu) (net 1) (status 1000000))
+  (segment (start 39 92) (end 27.6 103.4) (width 0.75) (layer F.Cu) (net 1) (status 1000000))
+  (segment (start 27.6 103.4) (end 27.6 105) (width 0.75) (layer F.Cu) (net 1) (status 1000000))
+  (segment (start 38 77) (end 38 80) (width 1) (layer F.Cu) (net 1) (status 1000000))
   (segment (start 32 89) (end 32 88.0625) (width 1) (layer B.Cu) (net 2) (status 30))
   (segment (start 35.5 92.5) (end 32 89) (width 1) (layer B.Cu) (net 2) (status 20))

Commit message: 04_14 fix1
Connections:
- C6 pad 2: +5V -> GND
Routing:
- net +5V: track 278.3 -> 274.1 mm
Changed lines of the file:
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@@
     (thickness 1.6)
     (drawings 4)
-    (tracks 364)
+    (tracks 362)
     (zones 0)
     (modules 62)
@@
     (fp_line (start -1.6 -0.8) (end -1.6 0.8) (layer B.Fab) (width 0.1))
     (pad 2 smd roundrect (at 1.4 0 90) (size 1.25 1.75) (layers B.Cu B.Paste B.Mask) (roundrect_rratio 0.2)
-      (net 5 +5V))
+      (net 1 GND))
     (pad 1 smd roundrect (at -1.4 0 90) (size 1.25 1.75) (layers B.Cu B.Paste B.Mask) (roundrect_rratio 0.2)
       (net 6 "Net-(C6-Pad1)"))
@@
   (via (at 51 108) (size 0.8) (drill 0.4) (layers F.Cu B.Cu) (net 1))
   (segment (start 58 101) (end 51 108) (width 1) (layer F.Cu) (net 1))
-  (segment (start 36 79.2) (end 36 79) (width 1) (layer F.Cu) (net 1))
-  (segment (start 36 79) (end 38 77) (width 1) (layer F.Cu) (net 1))
+  (segment (start 36 79.2) (end 36 79) (width 1) (layer F.Cu) (net 1) (status 30))
+  (segment (start 36 79) (end 38 77) (width 1) (layer F.Cu) (net 1) (status 10))
   (segment (start 38 77) (end 38 72) (width 1) (layer F.Cu) (net 1))
-  (segment (start 37.2 71.2) (end 36 71.2) (width 1) (layer F.Cu) (net 1))
+  (segment (start 37.2 71.2) (end 36 71.2) (width 1) (layer F.Cu) (net 1) (status 20))
   (segment (start 38 72) (end 37.2 71.2) (width 1) (layer F.Cu) (net 1))
-  (segment (start 38 80) (end 39 81) (width 0.75) (layer F.Cu) (net 1) (status 1000000))
-  (segment (start 39 81) (end 39 92) (width 0.75) (layer F.Cu) (net 1) (status 1000000))
-  (segment (start 39 92) (end 27.6 103.4) (width 0.75) (layer F.Cu) (net 1) (status 1000000))
-  (segment (start 27.6 103.4) (end 27.6 105) (width 0.75) (layer F.Cu) (net 1) (status 1000000))
-  (segment (start 38 77) (end 38 80) (width 1) (layer F.Cu) (net 1) (status 1000000))
+  (segment (start 38 80) (end 39 81) (width 0.75) (layer F.Cu) (net 1))
+  (segment (start 39 81) (end 39 92) (width 0.75) (layer F.Cu) (net 1))
+  (segment (start 39 92) (end 27.6 103.4) (width 0.75) (layer F.Cu) (net 1))
+  (segment (start 27.6 103.4) (end 27.6 105) (width 0.75) (layer F.Cu) (net 1) (status 20))
+  (segment (start 38 77) (end 38 80) (width 1) (layer F.Cu) (net 1))
   (segment (start 32 89) (end 32 88.0625) (width 1) (layer B.Cu) (net 2) (status 30))
   (segment (start 35.5 92.5) (end 32 89) (width 1) (layer B.Cu) (net 2) (status 20))
@@
   (segment (start 48.6 89.8) (end 48.62 89.78) (width 1) (layer B.Cu) (net 4) (status 30))
   (segment (start 45 89.8) (end 48.6 89.8) (width 1) (layer B.Cu) (net 4) (status 30))
-  (segment (start 52.4 90) (end 52 89.6) (width 1) (layer B.Cu) (net 5) (status 30))
-  (segment (start 56 90) (end 52.4 90) (width 1) (layer B.Cu) (net 5) (status 30))
   (segment (start 40.96 87.2) (end 41 87.24) (width 1) (layer B.Cu) (net 5) (status 30))
   (segment (start 37 87.2) (end 40.96 87.2) (width 1) (layer B.Cu) (net 5) (status 30))
@@
   (segment (start 59.5 95.5) (end 60.41 94.59) (width 1) (layer B.Cu) (net 29))
   (via (at 38 108) (size 0.8) (drill 0.4) (layers F.Cu B.Cu) (net 30))
-  (segment (start 36.4 105) (end 36.4 106.4) (width 0.75) (layer F.Cu) (net 30))
+  (segment (start 36.4 105) (end 36.4 106.4) (width 0.75) (layer F.Cu) (net 30) (status 10))
   (segment (start 36.4 106.4) (end 38 108) (width 0.75) (layer F.Cu) (net 30))
-  (segment (start 40.98 105.02) (end 41 105.02) (width 0.75) (layer B.Cu) (net 30))
-  (segment (start 38 108) (end 40.98 105.02) (width 0.75) (layer B.Cu) (net 30))
-  (segment (start 30.4 105) (end 33.6 105) (width 0.75) (layer F.Cu) (net 31))
+  (segment (start 40.98 105.02) (end 41 105.02) (width 0.75) (layer B.Cu) (net 30) (status 30))
+  (segment (start 38 108) (end 40.98 105.02) (width 0.75) (layer B.Cu) (net 30) (status 20))
+  (segment (start 30.4 105) (end 33.6 105) (width 0.75) (layer F.Cu) (net 31) (status 30))
   (zone (net 1) (net_name GND) (layer B.Cu) (hatch edge 0.508)
     (connect_pads (clearance 0.508))
