File: PCB KiCad/DRS CAN/DRS.kicad_pcb (KiCad board)
At the start: 2 copper layers, 38 parts, among them J1 Screw_Terminal_01x02, J2 Screw_Terminal_01x06, J3 Conn_02x03_Odd_Even, J4 Conn_01x03_Male, SW1 SW_Push, SW2 SW_Push, SW3 SW_Push, U1 AT90CAN32-16AU, U2 MCP2562-E-SN, U3 LM2596S-5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

Commit message: 04_14 CANv2
Parts:
- removed D6: D_Zener, Diode_SMD:D_SMB
- added D5: D_Schottky, Diode_SMD:D_SMB, F.Cu at (65.2, 96.2)
- added J5: Screw_Terminal_01x04, TerminalBlock_4Ucon:TerminalBlock_4Ucon_1x04_P3.50mm_Vertical, F.Cu at (89.6, 60.0)
- C1, C2: footprint Capacitor_SMD:C_0805_2012Metric -> Capacitor_SMD:C_1206_3216Metric
- J2: value Screw_Terminal_01x06 -> Screw_Terminal_01x02; footprint TerminalBlock_4Ucon:TerminalBlock_4Ucon_1x06_P3.50mm_Vertical -> TerminalBlock_4Ucon:TerminalBlock_4Ucon_1x02_P3.50mm_Vertical
- Y1: footprint Crystal:Crystal_SMD_HC49-SD_HandSoldering -> Crystal:Crystal_SMD_HC49-SD
- moved J3 97.5 mm to (110.9, 90.2)
- moved Y1 97.3 mm to (115.8, 74.4), turned to 270 degrees
- moved SW2 83.9 mm to (120.5, 63.7), turned to 180 degrees
- moved SW1 82.7 mm to (119.4, 84.6)
- moved J2 68.9 mm to (99.9, 91.4)
- moved C9 68.5 mm to (65.3, 89.0), turned to 270 degrees
- moved U1 67.2 mm to (99.4, 73.6), turned to 90 degrees
- moved R1 66.5 mm to (121.4, 89.2)
- moved C3 65.0 mm to (126.0, 84.6), turned to 90 degrees
- moved R2 62.5 mm to (127.2, 63.2), turned to 90 degrees
- moved SW3 60.7 mm to (120.5, 56.2)
- moved L3 58.0 mm to (76.0, 90.8)
- moved U3 57.7 mm to (72.5, 75.6), turned to 90 degrees
- moved J4 55.8 mm to (92.5, 90.8), turned to 270 degrees
- moved C2 52.5 mm to (119.6, 77.0), turned to 90 degrees
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Connections:
- C6 pad 1: Net-(C6-Pad1) -> GND
- C6 pad 2: +5V -> Net-(C6-Pad2)
- D1 pad 2: (no net) -> /LED
- J2 pad 1: +12V -> /PWM1
- J2 pad 2: /CANL -> /PWM2
- J4 pad 2: (no net) -> +5V
- L1 pad 2: Net-(C6-Pad1) -> Net-(C6-Pad2)
- U1 pad 10: (no net) -> /LED
- U1 pad 64: Net-(C6-Pad1) -> Net-(C6-Pad2)
Routing:
- net Net-(C2-Pad1): track 0.00 -> 16.1 mm
- net Net-(C1-Pad1): track 0.00 -> 16.1 mm
- net GND: track 0.00 -> 2.40 mm
Other:
- net class Default: trace_width 0.25 -> 0.5

Commit message: 05_05 v2
Skończony projekt testowy na at90can
Parts:
- L1: footprint Connector_PinSocket_2.54mm:PinSocket_1x02_P2.54mm_Vertical -> Inductor_SMD:L_1812_4532Metric
- moved J3 5.06 mm to (108.8, 85.6), turned to 0 degrees
- moved D4 4.25 mm to (66.4, 60.0), turned to 0 degrees
- moved J2 3.10 mm to (99.9, 94.5)
- moved J5 3.00 mm to (89.6, 57.0)
- moved D8 2.99 mm to (83.8, 69.0)
- moved R1 2.80 mm to (124.2, 89.2), turned to 180 degrees
- moved R9 2.37 mm to (83.8, 71.8)
- moved C8 1.25 mm to (114.0, 58.0), turned to 90 degrees
- moved R2 1.22 mm to (127.0, 64.4), turned to 270 degrees
- moved R3 1.22 mm to (127.0, 58.0), turned to 90 degrees
- moved F2 1.17 mm to (64.4, 68.8)
- moved SW3 1.02 mm to (120.5, 57.2), turned to 180 degrees
- moved D2 0.85 mm to (64.4, 76.6)
- moved L1 0.58 mm to (86.4, 86.0), turned to 0 degrees
- moved C9 0.28 mm to (65.0, 89.0)
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Connections:
- J5 pad 1: +12V -> /CANL
- J5 pad 2: /CANL -> /CANH
- J5 pad 3: /CANH -> +12V
Routing:
- net +5V: track 0.00 -> 218.0 mm, vias 0 -> 2
- net GND: track 2.40 -> 183.2 mm, vias 0 -> 9
- net /Button2: track 0.00 -> 49.3 mm, vias 0 -> 1
- net /RESET: track 0.00 -> 46.0 mm, vias 0 -> 1
- net /Button1: track 0.00 -> 40.5 mm, vias 0 -> 1
- net +12P: track 0.00 -> 38.0 mm
- net /MOSI: track 0.00 -> 35.1 mm, vias 0 -> 1
- net /CANH: track 0.00 -> 27.4 mm, vias 0 -> 1
- net /PWM1: track 0.00 -> 26.6 mm, vias 0 -> 1
- net +12V: track 0.00 -> 26.3 mm, vias 0 -> 1
- net /PWM2: track 0.00 -> 22.0 mm, vias 0 -> 1
- net /CANL: track 0.00 -> 19.2 mm, vias 0 -> 1
- net /MISO: track 0.00 -> 18.3 mm, vias 0 -> 1
- net Net-(D5-Pad1): track 0.00 -> 16.9 mm
- net /RXCAN: track 0.00 -> 12.5 mm
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- added copper zone on B.Cu, net GND
Other:
- board outline added: 70 x 46.5 mm
- board text added: "DRS V1 PUT Motorsport Eryk Miskiewicz"
