File: PCB KiCad/DRS CAN/V2/DRS.kicad_pcb (KiCad board)
At the start: 2 copper layers, 82.5 x 52.5 mm, 64 parts, among them J1 Screw_Terminal_01x04, J2 Screw_Terminal_01x03, J3 Conn_02x03_Odd_Even, J4 Screw_Terminal_01x03, SW1 SW_Push, SW2 SW_Push, SW3 SW_Push, U1 AT90CAN32-16AU, U2 MCP2562-E-SN, U3 AP1501-K5G-13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

Commit message: Adjustable voltage fix
Parts:
- added R14: 0R, Resistor_SMD:R_1206_3216Metric, B.Cu at (152.5, 83.5)
- added R15: 0R, Resistor_SMD:R_1206_3216Metric, B.Cu at (114.8, 74.5)
- added R16: 0R, Resistor_SMD:R_1206_3216Metric, B.Cu at (151.2, 79.4)
- added R17: 0R, Resistor_SMD:R_1206_3216Metric, B.Cu at (116.0, 78.2)
- moved C17 2.81 mm to (110.8, 80.5)
- moved C16 0.95 mm to (156.0, 77.2)
Connections:
- U3 pad 4: +5VP -> Net-(R14-Pad2)
- U4 pad 4: +5VL -> Net-(R15-Pad2)
Routing:
- net +5VP: track 58.8 -> 43.6 mm
- net +5VL: track 54.1 -> 41.8 mm
- net Net-(R14-Pad2): track 0.00 -> 12.0 mm
- net Net-(R15-Pad2): track 0.00 -> 11.2 mm
- net GND: track 526.3 -> 527.5 mm

Commit message: WersjaV2 PCB
Parts:
- added D13: BAT54S, Package_TO_SOT_SMD:SOT-23, B.Cu at (126.5, 90.2)
- added D14: BAT54S, Package_TO_SOT_SMD:SOT-23, B.Cu at (165.4, 64.6)
- added R18: 1k, Resistor_SMD:R_1206_3216Metric, B.Cu at (121.7, 89.2)
- added R19: 1k, Resistor_SMD:R_1206_3216Metric, B.Cu at (161.8, 63.8)
Connections:
- J2 pad 1: /PWM1 -> /Złącza/PWM1Out
- J4 pad 1: /PWM2 -> /Złącza/PWM2Out
Routing:
- net +5V: track 231.5 -> 262.3 mm, vias 4 -> 5
- net /Złącza/PWM1Out: track 0.00 -> 27.0 mm
- net /PWM1: track 23.9 -> 5.72 mm
- net GND: track 527.5 -> 540.8 mm
- net /Złącza/PWM2Out: track 0.00 -> 9.11 mm
- net /PWM2: track 64.1 -> 58.2 mm
Other:
- board text added: "DRS CAN V2 PUT Motorsport Eryk Miśkiewicz"
- board text removed: "DRS CAN V1 PUT Motorsport Eryk Miśkiewicz"
